File: bartonfirtop/bartonfirtop.kicad_pcb (KiCad board)
At the start: 2 copper layers, 100 x 100 mm, 28 parts, among them J1 12v Supply, J10 LED8, J11 LED9, J12 LED10, J13 LED11, J14 LED12, J15 LED13, J16 LED14, J17 LED15, J18 LED16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

Commit message: testing 16 LEDs on the control board
Connections:
- U4 pad 14: Net-(J19-Pin_1) -> Net-(J12-Pin_1)
- U4 pad 15: Net-(J19-Pin_3) -> Net-(J11-Pin_1)
- U4 pad 19: Net-(J12-Pin_1) -> Net-(J19-Pin_1)
- U4 pad 20: Net-(J11-Pin_1) -> Net-(J19-Pin_3)
Routing:
- net Net-(J19-Pin_1): track 57.2 -> 116.4 mm
- net Net-(J19-Pin_3): track 50.8 -> 109.4 mm
- net Net-(J11-Pin_1): track 105.6 -> 122.7 mm
- net Net-(J12-Pin_1): track 106.5 -> 115.1 mm
Changed lines of the file:
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@@
 			)
 		)
+		(sheetname "Root")
+		(sheetfile "bartonfirtop.kicad_sch")
 		(attr through_hole)
 		(fp_line
@@
 			(layers "*.Cu" "*.Mask")
 			(remove_unused_layers no)
-			(net 22 "Net-(J19-Pin_1)")
+			(net 16 "Net-(J12-Pin_1)")
 			(pinfunction "D22")
 			(pintype "tri_state")
@@
 			(layers "*.Cu" "*.Mask")
 			(remove_unused_layers no)
-			(net 23 "Net-(J19-Pin_3)")
+			(net 15 "Net-(J11-Pin_1)")
 			(pinfunction "D23")
 			(pintype "tri_state")
@@
 			(layers "*.Cu" "*.Mask")
 			(remove_unused_layers no)
-			(net 16 "Net-(J12-Pin_1)")
+			(net 22 "Net-(J19-Pin_1)")
 			(pinfunction "D34")
 			(pintype "tri_state")
@@
 			(layers "*.Cu" "*.Mask")
 			(remove_unused_layers no)
-			(net 15 "Net-(J11-Pin_1)")
+			(net 23 "Net-(J19-Pin_3)")
 			(pinfunction "D35")
 			(pintype "tri_state")
@@
 			)
 		)
+		(sheetname "Root")
+		(sheetfile "bartonfirtop.kicad_sch")
 		(attr through_hole)
 		(fp_rect
@@
 	)
 	(segment
-		(start 177 87)
-		(end 177 89)
+		(start 168.5 62.5)
+		(end 175 69)
 		(width 1)
 		(layer "B.Cu")
@@
 	)
 	(segment
-		(start 177.9 89.9)
-		(end 181 89.9)
+		(start 175 86.197056)
+		(end 172.997056 88.2)
 		(width 1)
 		(layer "B.Cu")
@@
 	)
 	(segment
-		(start 175 69)
-		(end 175 85)
+		(start 169.13 88.2)
+		(end 157.27 100.06)
 		(width 1)
 		(layer "B.Cu")
@@
 	)
 	(segment
-		(start 106 68.5)
-		(end 112.5 68.5)
+		(start 175 69)
+		(end 175 86.197056)
 		(width 1)
 		(layer "B.Cu")
@@
 	)
 	(segment
-		(start 168.5 62.5)
-		(end 175 69)
+		(start 106 68.5)
+		(end 112.5 68.5)
 		(width 1)
 		(layer "B.Cu")
@@
 	)
 	(segment
-		(start 134.5 55)
-		(end 142 55)
+		(start 157.27 100.06)
+		(end 155.6 100.06)
 		(width 1)
 		(layer "B.Cu")
@@
 	)
 	(segment
-		(start 175 85)
-		(end 177 87)
+		(start 134.5 55)
+		(end 142 55)
 		(width 1)
 		(layer "B.Cu")
@@
 	)
 	(segment
-		(start 177 89)
-		(end 177.9 89.9)
+		(start 142 55)
+		(end 144 57)
 		(width 1)
 		(layer "B.Cu")
@@
 	)
 	(segment
-		(start 142 55)
-		(end 144 57)
+		(start 112.5 68.5)
+		(end 124 57)
 		(width 1)
 		(layer "B.Cu")
@@
 	)
 	(segment
-		(start 112.5 68.5)
-		(end 124 57)
+		(start 172.997056 88.2)
+		(end 169.13 88.2)
 		(width 1)
 		(layer "B.Cu")
@@
 	)
 	(segment
-		(start 172.5 87)
-		(end 177.94 92.44)
+		(start 172.5 71)
+		(end 172.5 83.81)
 		(width 1)
 		(layer "B.Cu")
@@
 	)
 	(segment
-		(start 129.5 58)
-		(end 140.5 58)
+		(start 165.5 64)
+		(end 172.5 71)
 		(width 1)
 		(layer "B.Cu")
@@
 	)
 	(segment
-		(start 140.5 58)
-		(end 141.5 59)
+		(start 129.5 58)
+		(end 140.5 58)
 		(width 1)
 		(layer "B.Cu")
@@
 	)
 	(segment
-		(start 172.5 71)
-		(end 172.5 87)
+		(start 140.5 58)
+		(end 141.5 59)
 		(width 1)
 		(layer "B.Cu")
@@
 	)
 	(segment
-		(start 165.5 64)
-		(end 172.5 71)
+		(start 172.5 83.81)
+		(end 171.27 85.04)
 		(width 1)
 		(layer "B.Cu")
@@
 	)
 	(segment
-		(start 177.94 92.44)
-		(end 181 92.44)
+		(start 156.95 97.52)
+		(end 155.6 97.52)
 		(width 1)
 		(layer "B.Cu")
@@
 	)
 	(segment
+		(start 171.27 85.04)
+		(end 169.43 85.04)
+		(width 1)
+		(layer "B.Cu")
+		(net 16)
+	)
+	(segment
+		(start 169.43 85.04)
+		(end 156.95 97.52)
+		(width 1)
+		(layer "B.Cu")
+		(net 16)
+	)
+	(segment
 		(start 106 76.05)
 		(end 108.45 76.05)
@@
 	)
 	(segment
-		(start 150 97.5)
-		(end 150.02 97.52)
+		(start 183.04 146.32)
+		(end 183.04 106.67)
 		(width 1)
 		(layer "F.Cu")
@@
 	)
 	(segment
-		(start 150.02 97.52)
-		(end 155.6 97.52)
+		(start 183.04 106.67)
+		(end 179.02 102.65)
 		(width 1)
 		(layer "F.Cu")
@@
 	)
 	(segment
-		(start 130.42 138.58)
-		(end 139.5 129.5)
+		(start 178.39 92.5)
+		(end 178.45 92.44)
 		(width 1)
 		(layer "F.Cu")
@@
 	)
 	(segment
-		(start 130.42 141)
-		(end 130.42 138.58)
+		(start 178.39 94.27)
+		(end 178.39 92.5)
 		(width 1)
 		(layer "F.Cu")
@@
 	)
 	(segment
-		(start 139.5 108)
-		(end 150 97.5)
+		(start 178.45 92.44)
+		(end 181 92.44)
 		(width 1)
 		(layer "F.Cu")
@@
 	)
 	(segment
-		(start 139.5 129.5)
-		(end 139.5 108)
+		(start 179.02 94.9)
+		(end 178.39 94.27)
 		(width 1)
 		(layer "F.Cu")
@@
 	)
 	(segment
-		(start 152.94 100.06)
-		(end 155.6 100.06)
+		(start 181.97 147.39)
+		(end 183.04 146.32)
+		(width 1)
+		(layer "F.Cu")
+		(net 22)
+	)
+	(segment
+		(start 132.92 147.39)
+		(end 181.97 147.39)
+		(width 1)
+		(layer "F.Cu")
+		(net 22)
+	)
+	(segment
+		(start 130.42 144.89)
+		(end 132.92 147.39)
+		(width 1)
+		(layer "F.Cu")
+		(net 22)
+	)
+	(segment
+		(start 179.02 102.65)
+		(end 179.02 94.9)
+		(width 1)
+		(layer "F.Cu")
+		(net 22)
+	)
+	(segment
+		(start 130.42 141)
+		(end 130.42 144.89)
+		(width 1)
+		(layer "F.Cu")
+		(net 22)
+	)
+	(segment
+		(start 176.5 95.13)
+		(end 176.26 94.89)
+		(width 1)
+		(layer "F.Cu")
+		(net 23)
+	)
+	(segment
+		(start 176.26 94.89)
+		(end 176.26 90.37)
+		(width 1)
+		(layer "F.Cu")
+		(net 23)
+	)
+	(segment
+		(start 177.2 89.9)
+		(end 181 89.9)
+		(width 1)
+		(layer "F.Cu")
+		(net 23)
+	)
+	(segment
+		(start 177.8 106.32)
+		(end 177.8 97.02)
+		(width 1)
+		(layer "F.Cu")
+		(net 23)
+	)
+	(segment
+		(start 176.26 90.37)
+		(end 176.73 90.37)
 		(width 1)
 		(layer "F.Cu")
@@
 	(segment
 		(start 135.5 141)
-		(end 135.5 138.5)
+		(end 135.5 142.35)
+		(width 1)
+		(layer "F.Cu")
+		(net 23)
+	)
+	(segment
+		(start 180.78 122.87)
+		(end 180.78 109.3)
+		(width 1)
+		(layer "F.Cu")
+		(net 23)
+	)
+	(segment
+		(start 180.66 145.25)
+		(end 180.66 122.99)
+		(width 1)
+		(layer "F.Cu")
+		(net 23)
+	)
+	(segment
+		(start 180.78 109.3)
+		(end 177.8 106.32)
+		(width 1)
+		(layer "F.Cu")
+		(net 23)
+	)
+	(segment
+		(start 138.4 145.25)
+		(end 180.66 145.25)
+		(width 1)
+		(layer "F.Cu")
+		(net 23)
+	)
+	(segment
+		(start 176.73 90.37)
+		(end 177.2 89.9)
+		(width 1)
+		(layer "F.Cu")
+		(net 23)
+	)
+	(segment
+		(start 180.66 122.99)
+		(end 180.78 122.87)
 		(width 1)
 		(layer "F.Cu")
@@
 	)
 	(segment
-		(start 145 129)
-		(end 145 108)
+		(start 176.5 95.72)
+		(end 176.5 95.13)
 		(width 1)
 		(layer "F.Cu")
@@
 	)
 	(segment
-		(start 145 108)
-		(end 152.94 100.06)
+		(start 135.5 142.35)
+		(end 138.4 145.25)
 		(width 1)
 		(layer "F.Cu")
@@
 	)
 	(segment
-		(start 135.5 138.5)
-		(end 145 129)
+		(start 177.8 97.02)
+		(end 176.5 95.72)
 		(width 1)
 		(layer "F.Cu")
